Commit message: Fiddled with the urdf a bit NOTE : NEED TO CHECK ALL FILES FOR LOCAL setup commands (nvidia drivers etc)

File: src/line_follower/worlds/sim_robot.urdf (robot description, URDF)
Before this commit: robot line_follower_robot, 4 links, 3 joints
Links:
- added link camera_optical_frame
- added link caster_wheel, mass 0.05; collision sphere radius=0.015; visual sphere radius=0.015
- link base_link: mass 1.0 -> 0.85; geometry collision box size=0.14 0.12 0.04; visual box size=0.006 0.03 0.002
- link camera_link: mass None -> 0.05; geometry collision box size=0.03 0.04 0.03; visual box size=0.03 0.04 0.03
- link left_wheel: mass 0.2 -> 0.15; geometry collision cylinder length=0.03 radius=0.035; visual cylinder length=0.03 radius=0.035
- link right_wheel: mass 0.2 -> 0.15; geometry collision cylinder length=0.03 radius=0.035; visual cylinder length=0.03 radius=0.035
Joints:
- added joint camera_optical_joint: type fixed, parent camera_link, child camera_optical_frame, origin xyz=0 0 0 rpy=-1.5708 0 -1.5708
- added joint caster_joint: type fixed, parent base_link, child caster_wheel, origin xyz=0.055 0 -0.035 rpy=0 0 0
- joint camera_joint: origin xyz=0.1 0 0.08 rpy=0 1.5708 0 -> xyz=-0.02 0 0.12 rpy=0 0.44 0
- joint left_wheel_joint: origin xyz=0.0 0.12 -0.03 rpy=0 0 0 -> xyz=-0.04 0.085 -0.015 rpy=0 0 0
- joint right_wheel_joint: origin xyz=0.0 -0.12 -0.03 rpy=0 0 0 -> xyz=-0.04 -0.085 -0.015 rpy=0 0 0
