Commit message: Changed urdf

File: src/line_follower/worlds/line_follower_robot.urdf (robot description, URDF)
Before this commit: robot line_follower_robot, 6 links, 5 joints
Links:
- removed link rear_caster
- link base_link: mass 0.34 -> 0.40; geometry collision box size=0.122 0.14 0.003; visual box size=0.006 0.020 0.0157
- link front_caster: mass 0.005 -> 0.01; geometry collision sphere radius=0.01; visual cylinder length=0.019 radius=0.003
- link left_wheel: mass 0.03 -> 0.02; geometry collision cylinder length=0.019 radius=0.0215; visual cylinder length=0.019 radius=0.0215
- link right_wheel: mass 0.03 -> 0.02; geometry collision cylinder length=0.019 radius=0.0215; visual cylinder length=0.019 radius=0.0215
Joints:
- removed joint rear_caster_joint
- joint camera_joint: origin xyz=0.040 0 0.0975 rpy=0 1.15 0 -> xyz=0.048 0 0.0372 rpy=0 0.75 0
- joint front_caster_joint: origin xyz=0.025 0 -0.0275 rpy=0 0 0 -> xyz=0.04 0 -0.011 rpy=0 0 0
- joint left_wheel_joint: origin xyz=0 0.070 0 rpy=0 0 0 -> xyz=-0.035 0.0645 0 rpy=0 0 0
- joint right_wheel_joint: origin xyz=0 -0.070 0 rpy=0 0 0 -> xyz=-0.035 -0.0645 0 rpy=0 0 0

Commit message: Massive Changes to LOGIC and changed sdf , urdf ,setup , launch practically everything

File: src/line_follower/worlds/line_follower_robot.urdf (robot description, URDF)
Before this commit: robot line_follower_robot, 5 links, 4 joints
Joints:
- joint camera_joint: origin xyz=0.048 0 0.0372 rpy=0 0.75 0 -> xyz=0.028 0 0.0372 rpy=0 0.53 0

Commit message: PID Changes

File: src/line_follower/worlds/line_follower_robot.urdf (robot description, URDF)
Before this commit: robot line_follower_robot, 5 links, 4 joints
Joints:
- joint camera_joint: origin xyz=0.028 0 0.0372 rpy=0 0.53 0 -> xyz=0.028 0 0.0372 rpy=0 0.43 0
